Commit message: 阶段提交

File: src/data/objects/bin/bin.urdf (robot description, URDF)
Before this commit: robot plane, 1 links, 0 joints
Links:
- link planeLink: geometry collision box size=0.5 0.5 0; visual mesh filename=bin.obj scale=0.5 0.5 0

File: src/data/objects/tray/traybox.urdf (robot description, URDF)
Before this commit: robot tabletop, 1 links, 0 joints
Links:
- link base_link: mass 10 -> 1

File: src/data/pybullet_objects/tray/traybox.urdf (robot description, URDF)
Before this commit: robot tabletop, 1 links, 0 joints
Links:
- link base_link: mass 0 -> 1

File: src/data/robots/ur5/ur5.urdf (robot description, URDF)
Before this commit: robot universal_robot, 8 links, 7 joints
Links:
- removed link placeholder
- added link ee_link, mass .001; collision box size=0.001 0.001 0.001; visual box size=0.01 0.01 0.01
- link base_link: geometry collision mesh filename=collision/base.stl; visual mesh filename=visual/base.obj
- link forearm_link: geometry collision mesh filename=collision/forearm.stl; visual mesh filename=visual/forearm.obj
- link shoulder_link: geometry collision mesh filename=collision/shoulder.stl; visual mesh filename=visual/shoulder.obj
- link upper_arm_link: geometry collision mesh filename=collision/upperarm.stl; visual mesh filename=visual/upperarm.obj
- link wrist_1_link: geometry collision mesh filename=collision/wrist1.stl; visual mesh filename=visual/wrist1.obj
- link wrist_2_link: geometry collision mesh filename=collision/wrist2.stl; visual mesh filename=visual/wrist2.obj
- link wrist_3_link: geometry collision mesh filename=collision/wrist3.stl; visual mesh filename=visual/wrist3.obj
Joints:
- removed joint joint7
- added joint jointEE: type fixed, parent wrist_3_link, child ee_link, origin xyz=0.0 0.084 0.0 rpy=0.0 0.0 0.0
- joint joint1: limit lower=-3.14159265359 upper=3.14159265359 effort=150.0 velocity=3.15 -> lower=-6.28318530718 upper=6.28318530718 effort=150.0 velocity=3.15
- joint joint2: limit lower=-3.14159265359 upper=3.14159265359 effort=150.0 velocity=3.15 -> lower=-6.28318530718 upper=6.28318530718 effort=150.0 velocity=3.15; origin xyz=0.0 0.13585 0.0 rpy=0 0 0 -> xyz=0.0 0.13585 0.0 rpy=0.0 0.0 0.0
- joint joint4: limit lower=-3.14159265359 upper=3.14159265359 effort=28.0 velocity=3.2 -> lower=-6.28318530718 upper=6.28318530718 effort=28.0 velocity=3.2; origin xyz=0.0 0.0 0.39225 rpy=0.0 0 0.0 -> xyz=0.0 0.0 0.39225 rpy=0.0 0.0 0.0
- joint joint5: limit lower=-3.14159265359 upper=3.14159265359 effort=28.0 velocity=3.2 -> lower=-6.28318530718 upper=6.28318530718 effort=28.0 velocity=3.2
- joint joint6: limit lower=-3.14159265359 upper=3.14159265359 effort=28.0 velocity=3.2 -> lower=-6.28318530718 upper=6.28318530718 effort=28.0 velocity=3.2
