Commit message: 拆垛

File: src/data/cameras/camera3d.urdf (robot description, URDF)
Before this commit: robot canera3d, 2 links, 1 joints
Links:
- link base: geometry visual mesh filename=camera3d/camera.obj scale=1 1 1

File: src/data/end_effectors/suction/suction.urdf (robot description, URDF)
Before this commit: robot universal_robot, 3 links, 2 joints
Links:
- removed link base_7
- removed link link8
- removed link link_7
- added link 11, mass .01; collision mesh filename=base.obj; visual mesh filename=base.obj
- added link ee, mass .001; visual mesh filename=link1.obj
- added link ee_link; visual box size=0.01 0.01 0.01
Joints:
- removed joint joint8
- removed joint joint_7
- added joint joint_ee: type fixed, parent 11, child ee, origin xyz=0 0.07 0 rpy=0 0 0, limit lower=0.00 upper=0.01 effort=20 velocity=0.2
- added joint joint_placeholder: type fixed, parent placeholder, child 11, origin xyz=0.0 0.054 0.0 rpy=0 0.0 0.0, axis 0 -1 0
