Commit message: 模型更新

File: src/data/end_effectors/gripper/gripper.urdf (robot description, URDF)
Before this commit: robot robotiq_arg2f_85_model, 11 links, 10 joints
Links:
- added link placeholder; visual box size=0.01 0.01 0.01
- link left_inner_finger: geometry collision mesh filename=collision/robotiq_arg2f_85_inner_finger.dae scale=0.001 0.001 0.001; visual mesh filename=visual/robotiq_arg2f_85_inner_finger.dae scale=0.001 0.001 0.001
- link left_inner_knuckle: geometry collision mesh filename=collision/robotiq_arg2f_85_inner_knuckle.dae scale=0.001 0.001 0.001; visual mesh filename=visual/robotiq_arg2f_85_inner_knuckle.dae scale=0.001 0.001 0.001
- link left_outer_finger: geometry collision mesh filename=collision/robotiq_arg2f_85_outer_finger.dae scale=0.001 0.001 0.001; visual mesh filename=visual/robotiq_arg2f_85_outer_finger.dae scale=0.001 0.001 0.001
- link left_outer_knuckle: geometry collision mesh filename=collision/robotiq_arg2f_85_outer_knuckle.dae scale=0.001 0.001 0.001; visual mesh filename=visual/robotiq_arg2f_85_outer_knuckle.dae scale=0.001 0.001 0.001
- link right_inner_finger: geometry collision mesh filename=collision/robotiq_arg2f_85_inner_finger.dae scale=0.001 0.001 0.001; visual mesh filename=visual/robotiq_arg2f_85_inner_finger.dae scale=0.001 0.001 0.001
- link right_inner_knuckle: geometry collision mesh filename=collision/robotiq_arg2f_85_inner_knuckle.dae scale=0.001 0.001 0.001; visual mesh filename=visual/robotiq_arg2f_85_inner_knuckle.dae scale=0.001 0.001 0.001
- link right_outer_finger: geometry collision mesh filename=collision/robotiq_arg2f_85_outer_finger.dae scale=0.001 0.001 0.001; visual mesh filename=visual/robotiq_arg2f_85_outer_finger.dae scale=0.001 0.001 0.001
- link right_outer_knuckle: geometry collision mesh filename=collision/robotiq_arg2f_85_outer_knuckle.dae scale=0.001 0.001 0.001; visual mesh filename=visual/robotiq_arg2f_85_outer_knuckle.dae scale=0.001 0.001 0.001
- link robotiq_arg2f_base_link: geometry collision mesh filename=collision/robotiq_arg2f_base_link.stl; visual mesh filename=visual/robotiq_arg2f_85_base_link.dae scale=0.001 0.001 0.001
Joints:
- added joint joint_placeholder: type fixed, parent placeholder, child robotiq_arg2f_base_link, origin xyz=0.0 0.0 0.0 rpy=-1.57 0.0 0.0, axis 0 -1 0

Commit message: 增加模型

File: src/data/end_effectors/gripper/gripper.urdf (robot description, URDF)
Before this commit: robot robotiq_arg2f_85_model, 12 links, 11 joints
Links:
- added link ee_link
Joints:
- removed joint joint_placeholder
- added joint joint_ee: type fixed, parent robotiq_arg2f_base_link, child ee_link, origin xyz=0.0 0.0 0.15 rpy=3.14 0.0 0.0
- added joint joint_placeholder_second: type fixed, parent placeholder, child robotiq_arg2f_base_link, origin xyz=0.0 0.0 0.0 rpy=-1.57 0.0 0.0, axis 0 -1 0
- joint finger_joint: limit lower=0 upper=0.8 effort=1000 velocity=2.0 -> lower=0 upper=0.8757 effort=1000 velocity=2.0
- joint right_outer_knuckle_joint: limit lower=0 upper=0.81 effort=1000 velocity=2.0 -> lower=0 upper=0.8757 effort=1000 velocity=2.0

File: src/data/robots/ur5/ur5.urdf (robot description, URDF)
Before this commit: robot universal_robot, 8 links, 7 joints
Links:
- removed link ee_link
- added link link_placeholder, mass .001; collision box size=0.001 0.001 0.001; visual box size=0.01 0.01 0.01
Joints:
- removed joint jointEE
- added joint joint_placeholder_first: type fixed, parent wrist_3_link, child link_placeholder, origin xyz=0.0 0.084 0.0 rpy=0.0 0.0 0.0

Commit message: 阶段提交

File: src/data/end_effectors/gripper/gripper.urdf (robot description, URDF)
Before this commit: robot robotiq_arg2f_85_model, 13 links, 12 joints
Joints:
- joint joint_ee: origin xyz=0.0 0.0 0.15 rpy=3.14 0.0 0.0 -> xyz=0.0 0.0 0.14 rpy=3.14 0.0 0.0

File: src/data/workpieces/suction/suction.urdf (robot description, URDF)
Before this commit: robot a, 1 links, 0 joints
Links:
- link link_a: geometry collision mesh filename=a.obj scale=4 4 10; visual mesh filename=a.obj scale=4 4 10
